Commit message: Actualización del nodo u2d2 y archivos STL

File: urdf/arms.urdf (robot description, URDF)
Before this commit: robot arms, 12 links, 11 joints
Joints:
- removed joint Q1R1_Joint
- removed joint Q1R2_Joint
- removed joint Q1R3_Joint
- removed joint Q2R1_Joint
- removed joint Q2R2_Joint
- removed joint Q2R3_Joint
- removed joint Q3R1_Joint
- removed joint Q3R2_Joint
- removed joint Q3R3_Joint
- added joint 10_Joint: type continuous, parent World_Link, child L1R1_Link, origin xyz=0.175 0  0.0077 rpy=0 0 -3.1416, axis 0 0 1
- added joint 11_Joint: type continuous, parent L1R1_Link, child L2R1_Link, origin xyz=0 0 0.059 rpy=1.5708 0 0, axis 0 0 1
- added joint 12_Joint: type continuous, parent L2R1_Link, child L3R1_Link, origin xyz=0.0784 0 0 rpy=0 0 0, axis 0 0 1
- added joint 20_Joint: type continuous, parent AxR2_Link, child L1R2_Link, origin xyz=0.175 0  0.0077 rpy=0 0 -3.1416, axis 0 0 1
- added joint 21_Joint: type continuous, parent L1R2_Link, child L2R2_Link, origin xyz=0 0 0.059 rpy=1.5708 0 0, axis 0 0 1
- added joint 22_Joint: type continuous, parent L2R2_Link, child L3R2_Link, origin xyz=0.0784 0 0 rpy=0 0 0, axis 0 0 1
- added joint 30_Joint: type continuous, parent AxR3_Link, child L1R3_Link, origin xyz=0.175 0  0.0077 rpy=0 0 -3.1416, axis 0 0 1
- added joint 31_Joint: type continuous, parent L1R3_Link, child L2R3_Link, origin xyz=0 0 0.059 rpy=1.5708 0 0, axis 0 0 1
- added joint 32_Joint: type continuous, parent L2R3_Link, child L3R3_Link, origin xyz=0.0784 0 0 rpy=0 0 0, axis 0 0 1

Commit message: Actualización nodo U2D2 y IDs de los dynamixel

File: urdf/arms.urdf (robot description, URDF)
Before this commit: robot arms, 12 links, 11 joints
Joints:
- removed joint 10_Joint
- removed joint 20_Joint
- removed joint 30_Joint
- added joint 13_Joint: type continuous, parent AxR3_Link, child L1R3_Link, origin xyz=0.175 0  0.0077 rpy=0 0 -3.1416, axis 0 0 1
- added joint 23_Joint: type continuous, parent L1R3_Link, child L2R3_Link, origin xyz=0 0 0.059 rpy=1.5708 0 0, axis 0 0 1
- added joint 33_Joint: type continuous, parent L2R3_Link, child L3R3_Link, origin xyz=0.0784 0 0 rpy=0 0 0, axis 0 0 1
- joint 11_Joint: child L2R1_Link -> L1R1_Link; origin xyz=0 0 0.059 rpy=1.5708 0 0 -> xyz=0.175 0  0.0077 rpy=0 0 -3.1416; parent L1R1_Link -> World_Link
- joint 12_Joint: child L3R1_Link -> L1R2_Link; origin xyz=0.0784 0 0 rpy=0 0 0 -> xyz=0.175 0  0.0077 rpy=0 0 -3.1416; parent L2R1_Link -> AxR2_Link
- joint 21_Joint: child L2R2_Link -> L2R1_Link; parent L1R2_Link -> L1R1_Link
- joint 22_Joint: child L3R2_Link -> L2R2_Link; origin xyz=0.0784 0 0 rpy=0 0 0 -> xyz=0 0 0.059 rpy=1.5708 0 0; parent L2R2_Link -> L1R2_Link
- joint 31_Joint: child L2R3_Link -> L3R1_Link; origin xyz=0 0 0.059 rpy=1.5708 0 0 -> xyz=0.0784 0 0 rpy=0 0 0; parent L1R3_Link -> L2R1_Link
- joint 32_Joint: child L3R3_Link -> L3R2_Link; parent L2R3_Link -> L2R2_Link

Commit message: Se actualizaron los nodos para la versión virtual

File: urdf/arms.urdf (robot description, URDF)
Before this commit: robot arms, 12 links, 11 joints
Joints:
- removed joint 11_Joint
- removed joint 12_Joint
- removed joint 13_Joint
- removed joint 21_Joint
- removed joint 22_Joint
- removed joint 23_Joint
- removed joint 31_Joint
- removed joint 32_Joint
- removed joint 33_Joint
- added joint dxl_11: type continuous, parent World_Link, child L1R1_Link, origin xyz=0.175 0  0.0077 rpy=0 0 -3.1416, axis 0 0 1
- added joint dxl_12: type continuous, parent AxR2_Link, child L1R2_Link, origin xyz=0.175 0  0.0077 rpy=0 0 -3.1416, axis 0 0 1
- added joint dxl_13: type continuous, parent AxR3_Link, child L1R3_Link, origin xyz=0.175 0  0.0077 rpy=0 0 -3.1416, axis 0 0 1
- added joint dxl_21: type continuous, parent L1R1_Link, child L2R1_Link, origin xyz=0 0 0.059 rpy=1.5708 0 0, axis 0 0 1
- added joint dxl_22: type continuous, parent L1R2_Link, child L2R2_Link, origin xyz=0 0 0.059 rpy=1.5708 0 0, axis 0 0 1
- added joint dxl_23: type continuous, parent L1R3_Link, child L2R3_Link, origin xyz=0 0 0.059 rpy=1.5708 0 0, axis 0 0 1
- added joint dxl_31: type continuous, parent L2R1_Link, child L3R1_Link, origin xyz=0.0784 0 0 rpy=0 0 0, axis 0 0 1
- added joint dxl_32: type continuous, parent L2R2_Link, child L3R2_Link, origin xyz=0.0784 0 0 rpy=0 0 0, axis 0 0 1
- added joint dxl_33: type continuous, parent L2R3_Link, child L3R3_Link, origin xyz=0.0784 0 0 rpy=0 0 0, axis 0 0 1
